File: hardware/hd-speccys-prototype/hd-speccys-prototype.kicad_pcb (KiCad board)
At the start: 2 copper layers, 148 x 104.5 mm, 20 parts, among them J1 PI_ZERO_2x20, J3 ULA_SOCKET_02x20, J4 Conn_01x03_Pin, J5 POWER 9-20VDC, U1 74LS30, U4 TSR_1-2450, U5 74HC244, U6 74HC244

Commit message: hw: schematic updates
Routing:
- net Net-(J3-/WR): track 48.8 -> 54.8 mm
Changed lines of the file:
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@@
   (segment (start 90.17 90.805) (end 91.0375 89.9375) (width 0.25) (layer "F.Cu") (net 50))
   (segment (start 114.7025 100.0975) (end 114.935 100.33) (width 0.25) (layer "F.Cu") (net 50))
+  (segment (start 119.4775 105.1775) (end 120.6025 106.3025) (width 0.25) (layer "F.Cu") (net 50))
+  (segment (start 120.6025 101.2225) (end 119.4775 102.3475) (width 0.25) (layer "F.Cu") (net 50))
   (segment (start 91.0375 89.9375) (end 95.6525 89.9375) (width 0.25) (layer "F.Cu") (net 50))
+  (segment (start 119.4775 102.3475) (end 119.4775 105.1775) (width 0.25) (layer "F.Cu") (net 50))
   (via (at 107.95 98.425) (size 0.8) (drill 0.4) (layers "F.Cu" "B.Cu") (net 50))
   (via (at 114.935 100.33) (size 0.8) (drill 0.4) (layers "F.Cu" "B.Cu") (net 50))
