File: hardware/hd-speccys-1_0a/hd-speccys.kicad_sch (KiCad schematic)
At the start: 52 parts, among them J1 9-20VDC, J2 PI_ZERO, J3 ULA_SOCKET, J4 ULA_ZX, J5 UART, J6 Debug_Data, J7 Debug_Ctrl, J8 PWR_OUT, U1 74LS541, U2 74LS541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

Commit message: hw: board updates
Parts:
- J1: value 9-20VDC -> POWER 9-20VDC
- J6, J7, J8: now in the parts list
- U4: footprint Converter_DCDC:Converter_DCDC_Murata_OKI-78SR_Horizontal -> Converter_DCDC:Converter_DCDC_TRACO_TSR-1_THT
Changed lines of the file:
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@@
       (effects (font (size 1.27 1.27)))
     )
-    (property "Footprint" "Converter_DCDC:Converter_DCDC_Murata_OKI-78SR_Horizontal" (at 48.26 184.15 0)
+    (property "Footprint" "Converter_DCDC:Converter_DCDC_TRACO_TSR-1_THT" (at 48.26 184.15 0)
       (effects (font (size 1.27 1.27) italic) (justify left) hide)
     )
@@
   )
   (symbol (lib_id "Connector:Conn_01x11_Pin") (at 179.07 100.33 0) (mirror y) (unit 1)
-    (in_bom no) (on_board no) (dnp no)
+    (in_bom yes) (on_board yes) (dnp no)
     (property "Reference" "J6" (at 181.61 83.82 0)
       (effects (font (size 1.27 1.27)))
@@
   )
   (symbol (lib_id "Connector:Conn_01x06_Pin") (at 207.01 83.82 0) (mirror y) (unit 1)
-    (in_bom no) (on_board no) (dnp no)
+    (in_bom yes) (on_board yes) (dnp no)
     (property "Reference" "J7" (at 208.28 95.25 0)
       (effects (font (size 1.27 1.27)))
@@
   )
   (symbol (lib_name "Conn_01x03_Pin_1") (lib_id "Connector:Conn_01x03_Pin") (at 68.58 30.48 0) (unit 1)
-    (in_bom no) (on_board no) (dnp no)
+    (in_bom yes) (on_board yes) (dnp no)
     (property "Reference" "J8" (at 66.04 21.59 0)
       (effects (font (size 1.27 1.27)))
@@
       (effects (font (size 1.27 1.27)))
     )
-    (property "Value" "9-20VDC" (at 24.13 171.45 0)
-      (effects (font (size 1.27 1.27)))
-    )
+    (property "Value" "POWER 9-20VDC" (at 24.13 171.45 0)
+      (effects (font (size 1.27 1.27)))
+    )
