File: hardware/hd-speccys-1_0a/hd-speccys-1_0a.kicad_pcb (KiCad board)
At the start: 2 copper layers, 143.5 x 68.6 mm, 44 parts, among them J1 9-20VDC, J2 PI_ZERO, J3 ULA_SOCKET, J4 ULA_ZX, J5 UART, U1 74LS541, U2 74LS541, U3 74LS10, U4 TSR_1-2450, U5 74AHC1G32

Commit message: hw: 1.0a and 1.0b PCBs laid out
Parts:
- added Q1: 2N3904, Package_TO_SOT_THT:TO-92_Inline, F.Cu at (199.7, 71.4)
- added R20: 100R, Resistor_SMD:R_0603_1608Metric_Pad0.98x0.95mm_HandSolder, F.Cu at (203.0, 71.4)
- added R29: 4K7, Resistor_SMD:R_0603_1608Metric_Pad0.98x0.95mm_HandSolder, F.Cu at (195.6, 69.7)
- added R33: 1k2, Resistor_SMD:R_0603_1608Metric_Pad0.98x0.95mm_HandSolder, F.Cu at (193.6, 69.7)
- J1: footprint Connector_PinHeader_2.54mm:PinHeader_1x02_P2.54mm_Horizontal -> Connector_PinHeader_2.54mm:PinHeader_1x04_P2.54mm_Horizontal
- R31: value R -> 1K
Connections:
- J2 pad 27: unconnected-(J2-SA5_(GPIO0)-Pad27) -> Net-(J2-SA5_(GPIO0))
Routing:
- net Net-(J2-SA5_(GPIO0)): track 0.00 -> 95.3 mm, vias 0 -> 5
- net GND: track 310.8 -> 359.7 mm, vias 23 -> 22
- net VDD: track 147.5 -> 155.2 mm
- net Net-(Q1-B): track 0.00 -> 6.68 mm
- net Net-(J3-/CAS): track 107.8 -> 113.1 mm, vias 2 -> 3
- net Net-(J3-/WR): track 106.4 -> 111.5 mm, vias 2 -> 3
- net Net-(J3-/RD): track 69.0 -> 73.6 mm, vias 0 -> 1
- net Net-(Q1-C): track 0.00 -> 4.57 mm
- net Net-(J3-/DRAMWE): track 68.1 -> 72.2 mm, vias 0 -> 1
- net Net-(J3-A0): track 67.2 -> 71.0 mm, vias 0 -> 1
- net Net-(J3-A1): track 64.8 -> 68.6 mm, vias 0 -> 1
- net Net-(J3-A2): track 63.0 -> 66.3 mm, vias 0 -> 1
- net Net-(J1-RESET): track 0.00 -> 2.85 mm
- net Net-(J1-VCC): track 37.6 -> 40.1 mm
- net Net-(J3-MIC_TAPE): track 169.7 -> 170.5 mm
Other:
- board text added: "+9V"
- board text added: "GND"
- board text added: "HD-SPECCYS Issue 2, Rev 1.0a © 2023 RA SEWELL"
- board text added: "RESET"
- board text added: "RXD"
- board text added: "TXD"
- board text removed: "HD-SPECCYS Issue 2, Rev 0.1a © 2023 RA SEWELL"
