File: hardware/hd-speccys-1_0a/hd-speccys-1_0a.kicad_sch (KiCad schematic)
At the start: 46 parts, among them J1 9-20VDC, J2 PI_ZERO, J3 ULA_SOCKET, J4 ULA_ZX, J5 UART, J6 Debug_Data, J7 Debug_Ctrl, J8 PWR_OUT, U1 74LS541, U2 74LS541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

Commit message: hw: 1.0a and 1.0b PCBs laid out
Parts:
- removed J1: 9-20VDC, Connector_PinHeader_2.54mm:PinHeader_1x02_P2.54mm_Horizontal, symbol Connector:Conn_01x02_Pin
- added J1: 9-20VDC, Connector_PinHeader_2.54mm:PinHeader_1x04_P2.54mm_Horizontal, symbol Connector:Conn_01x04_Pin
- added Q1: 2N3904, Package_TO_SOT_THT:TO-92_Inline, symbol Transistor_BJT:2N3904
- added R20: 100R, Resistor_SMD:R_0603_1608Metric_Pad0.98x0.95mm_HandSolder, symbol Device:R
- added R29: 4K7, Resistor_SMD:R_0603_1608Metric_Pad0.98x0.95mm_HandSolder, symbol Device:R
- added R33: 1k2, Resistor_SMD:R_0603_1608Metric_Pad0.98x0.95mm_HandSolder, symbol Device:R
- R31: value R -> 1K
Connections:
- net GND: now also J1.2 (GND), Q1.1 (E), R29.2
- net at U4.1 (Vin): now also J1.1 (VCC)
- net at J2.27 (SA5_(GPIO0)): now also R33.1
- new net: J1.4 (RESET), R20.1
- new net: Q1.2 (B), R29.1, R33.2
- new net: Q1.3 (C), R20.2
Other:
- note added: "TODO: Define these values based on testing TODO: Check grounding (don't connect wrong GNDs together)"
- note removed: "TODO: Define these values based on testing TODO: Add reset control TODO: Add +/- terminals to silkscreen TODO: Check grounding (don't connect wrong GNDs together)"
- moved on the sheet: J8, R1, U3A, U3B, U3C, U4
