File: hardware/hd-speccys/hd-speccys.kicad_pcb (KiCad board)
At the start: 2 copper layers, 68.6 x 68.6 mm, 55 parts, among them J1 POWER 9-20VDC, J2 PI_ZERO_2x20, J3 ULA_SOCKET_02x20, J4 ULA_ZX_02x20, J5 UART, J6 Debug_Data, J7 Debug_Ctrl, U1 74LS541, U2 74LS541, U3 74HC00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

Commit message: hw: schematic updates
Parts:
- removed C5: C, Capacitor_SMD:C_0603_1608Metric_Pad1.08x0.95mm_HandSolder
- removed R33, R34, R35: R, Resistor_SMD:R_0603_1608Metric_Pad0.98x0.95mm_HandSolder
- U3: value 74HC00 -> 74LS10
- U5: value 74HC00 -> 74AHC1G32; footprint Package_SO:TSSOP-14_4.4x5mm_P0.65mm -> Package_TO_SOT_SMD:SOT-353_SC-70-5_Handsoldering
- moved R1 25.7 mm to (102.2, 56.5)
- moved U5 13.9 mm to (93.3, 62.2)
- moved U3 2.59 mm to (93.0, 54.6)
- moved C4 2.56 mm to (95.2, 50.5)
- moved R29 0.08 mm to (102.2, 60.3)
- moved R30 0.08 mm to (102.2, 58.4)
Connections:
- J7 pad 1: Net-(J2-GPIO27) -> Net-(J2-SD16_(DREQ))
- J7 pad 2: Net-(J2-SD1) -> Net-(J7-Pin_2)
- J7 pad 4: Net-(J2-SD0) -> Net-(J2-SD1)
- J7 pad 5: Net-(J7-Pin_5) -> Net-(J2-SD0)
- J7 pad 6: Net-(J7-Pin_6) -> Net-(J2-GPIO27)
- R1 pad 1: Net-(U1-A0) -> Net-(J2-SD16_(DREQ))
- R1 pad 2: Net-(J3-/IOREQ) -> Net-(R1-Pad2)
- R29 pad 2: Net-(J7-Pin_5) -> Net-(J7-Pin_2)
- R30 pad 2: Net-(J7-Pin_6) -> Net-(R30-Pad2)
- U1 pad 18: Net-(U1-Y0) -> unconnected-(U1-Y0-Pad18)
- U1 pad 2: Net-(U1-A0) -> GND
- U3 pad 10: Net-(J7-Pin_6) -> Net-(U3-Pad10)
- U3 pad 11: Net-(R33-Pad2) -> Net-(U3-Pad10)
- U3 pad 12: Net-(U3-Pad12) -> Net-(R30-Pad2)
- U3 pad 13: Net-(U3-Pad12) -> Net-(U1-Y7)
- U3 pad 2: Net-(U1-Y5) -> Net-(U1-Y3)
- U3 pad 3: Net-(J7-Pin_5) -> Net-(R30-Pad2)
- U3 pad 4: Net-(U1-Y0) -> Net-(R30-Pad2)
- U3 pad 5: Net-(U1-Y3) -> Net-(R30-Pad2)
- U3 pad 6: Net-(J7-Pin_6) -> Net-(U3-Pad10)
- U3 pad 8: Net-(U3-Pad12) -> Net-(R1-Pad2)
- U3 pad 9: Net-(J7-Pin_6) -> Net-(U3-Pad10)
- U5 pad 1: Net-(R33-Pad2) -> Net-(U1-Y1)
- U5 pad 2: Net-(R33-Pad2) -> Net-(U1-Y5)
- U5 pad 3: Net-(U5-Pad3) -> GND
- U5 pad 4: Net-(U5-Pad3) -> Net-(J7-Pin_2)
- U5 pad 5: Net-(U5-Pad3) -> VDDA
Routing:
- net Net-(J7-Pin_6): track 35.4 -> 0.00 mm, vias 2 -> 0
- net Net-(U1-A0): track 32.0 -> 0.00 mm
- net Net-(J7-Pin_5): track 27.7 -> 0.00 mm, vias 5 -> 0
- net Net-(R33-Pad2): track 25.1 -> 0.00 mm
- net Net-(U1-Y7): track 8.47 -> 29.6 mm, vias 0 -> 4
- net Net-(R30-Pad2): track 0.00 -> 19.4 mm, vias 0 -> 2
- net Net-(U1-Y0): track 18.8 -> 0.00 mm, vias 2 -> 0
- net Net-(J2-GPIO27): track 39.7 -> 21.4 mm
- net Net-(R34-Pad2): track 17.2 -> 0.00 mm
- net Net-(J7-Pin_2): track 0.00 -> 17.1 mm, vias 0 -> 2
- net GND: track 112.0 -> 101.5 mm
- net Net-(U1-Y1): track 23.0 -> 32.9 mm, vias 2 -> 0
- net Net-(R35-Pad2): track 8.94 -> 0.00 mm
- net Net-(U5-Pad12): track 7.86 -> 0.00 mm, vias 2 -> 0
- net Net-(U3-Pad12): track 7.77 -> 0.00 mm, vias 2 -> 0
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Other:
- board text added: "HD-SPECCYS Rev 0.1a © 2023 RA SEWELL, ERIC SEWELL"

Commit message: hw: Finished silkscreen
Parts:
- added J8: GND, Connector_PinHeader_2.54mm:PinHeader_1x01_P2.54mm_Vertical, F.Cu at (89.4, 47.5)
- J2: value PI_ZERO_2x20 -> PI_ZERO
- J3: value ULA_SOCKET_02x20 -> ULA_SOCKET
- J4: value ULA_ZX_02x20 -> ULA_ZX
Routing:
- net GND: track 101.5 -> 116.0 mm, vias 13 -> 14
- net VDDA: track 99.2 -> 100.0 mm
Other:
- board text added: "/CAS"
- board text added: "/INT"
- board text added: "/IOREQ"
- board text added: "/IO_WR"
- board text added: "/WR"
- board text added: "D0"
- board text added: "D1"
- board text added: "D2"
- board text added: "D3"
- board text added: "D4"
- board text added: "D5"
- board text added: "D6"
- board text added: "D7"
- board text added: "DREQ"
- board text added: "GND"
- board text added: "RXD0"
- board text added: "TXD0"

Commit message: hw: board updates
Parts:
- removed J6: Debug_Data, Connector_PinHeader_2.54mm:PinHeader_1x08_P2.54mm_Vertical
- removed J7: Debug_Ctrl, Connector_PinHeader_2.54mm:PinHeader_1x06_P2.54mm_Vertical
- removed J8: GND, Connector_PinHeader_2.54mm:PinHeader_1x01_P2.54mm_Vertical
- added ?: , , F.Cu at (85.3, 82.2)
- J1: value POWER 9-20VDC -> 9-20VDC
- U4: footprint Converter_DCDC:Converter_DCDC_TRACO_TSR-1_THT -> Converter_DCDC:Converter_DCDC_Murata_OKI-78SR_Horizontal
- moved J3 151.4 mm to (215.9, 77.5), turned to -90 degrees
- moved J4 92.4 mm to (149.9, 80.0)
- moved U4 79.4 mm to (177.0, 66.3)
- moved J1 77.1 mm to (192.4, 70.5)
- moved J5 53.3 mm to (75.6, 89.5), turned to 180 degrees
- moved R16 53.0 mm to (123.3, 63.5), turned to 0 degrees
- moved R15 51.4 mm to (123.3, 65.2), turned to 0 degrees
- moved R14 50.1 mm to (123.3, 66.8), turned to 0 degrees
- moved R13 48.9 mm to (123.3, 68.5), turned to 0 degrees
- moved R12 48.0 mm to (123.3, 70.1), turned to 0 degrees
- moved R11 47.4 mm to (123.3, 71.8), turned to 0 degrees
- moved R2 47.0 mm to (117.8, 80.6), turned to 0 degrees
- moved R10 47.0 mm to (123.3, 73.4), turned to 0 degrees
- moved R9 46.8 mm to (123.3, 75.1), turned to 0 degrees
- moved R3 45.4 mm to (117.8, 79.0), turned to 0 degrees
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Connections:
- J2 pad 31: unconnected-(J2-SOE_SE-Pad31) -> Net-(J2-SOE_SE)
Routing:
- net GND: track 116.0 -> 359.6 mm, vias 14 -> 25
- net VDD: track 21.8 -> 157.0 mm, vias 0 -> 4
- net Net-(J3-/INT): track 10.5 -> 138.3 mm, vias 0 -> 1
- net Net-(J3-D0): track 19.5 -> 145.3 mm, vias 0 -> 1
- net Net-(J3-MIC_TAPE): track 40.1 -> 150.4 mm, vias 3 -> 8
- net Net-(J3-D3): track 10.8 -> 116.7 mm
- net Net-(J3-D2): track 19.4 -> 121.6 mm
- net Net-(J3-D1): track 28.2 -> 122.3 mm, vias 0 -> 1
- net Net-(J3-D4): track 19.3 -> 113.2 mm
- net Net-(J3-D5): track 23.7 -> 111.1 mm
- net Net-(J3-D6): track 28.8 -> 110.2 mm
- net Net-(J3-/IOREQ): track 15.7 -> 96.6 mm, vias 2 -> 3
- net Net-(J3-D7): track 33.9 -> 109.3 mm
- net Net-(J3-/CAS): track 31.7 -> 105.2 mm, vias 0 -> 3
- net Net-(J3-/WR): track 32.7 -> 104.7 mm, vias 0 -> 3
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Other:
- board size 68.6 x 68.6 mm -> 143.5 x 68.6 mm
- board text added: "HD-SPECCYS Issue 2, Rev 0.1a © 2023 RA SEWELL"
- board text added: "VOL"
- board text removed: "/CAS"
- board text removed: "/INT"
- board text removed: "/IOREQ"
- board text removed: "/IO_WR"
- board text removed: "/WR"
- board text removed: "D0"
- board text removed: "D1"
- board text removed: "D2"
- board text removed: "D3"
- board text removed: "D4"
- board text removed: "D5"
- board text removed: "D6"
- board text removed: "D7"
- board text removed: "DREQ"
- board text removed: "GND"
- board text removed: "HD-SPECCYS Rev 0.1a © 2023 RA SEWELL, ERIC SEWELL"
- board text removed: "RXD0"
- board text removed: "TXD0"

Commit message: hw: PCB modifications - route between ULA pins and socket efficiently
Parts:
- removed C1: 100nF, Capacitor_SMD:C_0603_1608Metric_Pad1.08x0.95mm_HandSolder
- removed D1, D2, D3: 1N4148, Diode_SMD:D_SOD-323_HandSoldering
- removed R20, R29: R, Resistor_SMD:R_0603_1608Metric_Pad0.98x0.95mm_HandSolder
- moved J1 14.6 mm to (205.8, 64.8)
- moved R31 11.9 mm to (90.9, 77.0), turned to 0 degrees
Connections:
- J2 pad 26: Net-(D3-A) -> Net-(J2-SWE_SRW_(GPIO7))
- R21 pad 1: Net-(J2-SD15) -> Net-(J2-SD8)
- R22 pad 1: Net-(J2-SD14) -> Net-(J2-SD9)
- R23 pad 1: Net-(J2-SD13) -> Net-(J2-SD10)
- R24 pad 1: Net-(J2-SD12) -> Net-(J2-SD11)
- R25 pad 1: Net-(J2-SD11) -> Net-(J2-SD12)
- R26 pad 1: Net-(J2-SD10) -> Net-(J2-SD13)
- R27 pad 1: Net-(J2-SD9) -> Net-(J2-SD14)
- R28 pad 1: Net-(J2-SD8) -> Net-(J2-SD15)
- R31 pad 2: Net-(C1-Pad1) -> Net-(J3-MIC_TAPE)
- R32 pad 1: Net-(D1-K) -> Net-(J2-SWE_SRW_(GPIO7))
- U1 pad 11: Net-(U1-Y7) -> Net-(J2-GPIO27)
- U3 pad 13: Net-(U1-Y7) -> Net-(J2-GPIO27)
- U5 pad 4: Net-(J7-/IO_WR) -> Net-(J2-GPIO26)
Routing:
- net Net-(J3-/IOREQ): track 96.6 -> 168.6 mm, vias 3 -> 4
- net Net-(J2-SWE_SRW_(GPIO7)): track 0.00 -> 54.8 mm
- net Net-(J3-D7): track 109.3 -> 163.2 mm, vias 1 -> 2
- net GND: track 359.6 -> 310.8 mm, vias 25 -> 23
- net Net-(J3-D6): track 110.2 -> 157.2 mm, vias 1 -> 2
- net Net-(D3-A): track 41.9 -> 0.00 mm
- net Net-(J3-/CPU): track 38.1 -> 75.9 mm, vias 1 -> 2
- net Net-(J3-D5): track 111.1 -> 143.7 mm, vias 1 -> 2
- net Net-(U1-Y7): track 29.9 -> 0.00 mm, vias 4 -> 0
- net Net-(J2-GPIO27): track 26.5 -> 56.1 mm, vias 2 -> 6
- net Net-(J3-D4): track 113.2 -> 135.2 mm, vias 1 -> 2
- net Net-(J3-MIC_TAPE): track 150.4 -> 169.7 mm, vias 8 -> 4
- net Net-(J3-KB4): track 38.1 -> 56.3 mm, vias 1 -> 2
- net Net-(J3-D3): track 116.7 -> 133.9 mm, vias 1 -> 2
- net Net-(J3-/INT): track 138.3 -> 123.1 mm
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Other:
- outline, holes or cut-outs redrawn
