File: hardware/hd-speccys-1_0b/hd-speccys-1_0b.kicad_pcb (KiCad board)
At the start: 2 copper layers, 143.5 x 68.6 mm, 42 parts, among them J1 9-20VDC, J2 PI_ZERO, J3 ULA_SOCKET, J4 ULA_ZX, J5 UART, Q1 2N3906, U3 74LS10, U4 TSR_1-2450, U5 74AHC1G32

Commit message: hw: 1.0a and 1.0b PCBs laid out
Parts:
- removed Q1: 2N3906, Package_TO_SOT_THT:TO-92_Inline
- added Q2: 2N3904, Package_TO_SOT_THT:TO-92_Inline, F.Cu at (199.7, 71.4)
- added R20: 4K7, Resistor_SMD:R_0603_1608Metric_Pad0.98x0.95mm_HandSolder, F.Cu at (195.5, 69.6)
- R2: value R -> 100R
- R3: value R -> 1k2
- moved R2 6.37 mm to (203.0, 71.5), turned to 90 degrees
- moved R3 2.44 mm to (193.5, 69.6)
Connections:
- R2 pad 1: Net-(Q1-C) -> Net-(J1-RESET)
- R2 pad 2: GND -> Net-(Q2-C)
Routing:
- net GND: track 503.2 -> 521.2 mm
- net Net-(Q2-C): track 0.00 -> 4.41 mm
- net Net-(J1-RESET): track 6.73 -> 2.81 mm
- net Net-(Q1-C): track 3.21 -> 0.00 mm
- net Net-(Q2-B): track 4.06 -> 6.76 mm
- net Net-(J3-/IOREQ): track 174.6 -> 173.7 mm
- net Net-(J3-D7): track 162.0 -> 161.5 mm
Other:
- board text added: "+9V"
- board text added: "GND"
- board text added: "RESET"
- board text added: "RXD"
- board text added: "TXD"
