File: hardware/hd-speccys-1_0b/hd-speccys-1_0b.kicad_sch (KiCad schematic)
At the start: 44 parts, among them J1 9-20VDC, J2 PI_ZERO, J3 ULA_SOCKET, J4 ULA_ZX, J5 UART, J6 Debug_Data, J7 Debug_Ctrl, J8 PWR_OUT, Q1 2N3906, U3 74LS10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

Commit message: hw: 1.0a and 1.0b PCBs laid out
Parts:
- removed Q1: 2N3906, Package_TO_SOT_THT:TO-92_Inline, symbol Transistor_BJT:2N3906
- added Q2: 2N3904, Package_TO_SOT_THT:TO-92_Inline, symbol Transistor_BJT:2N3904
- added R20: 4K7, Resistor_SMD:R_0603_1608Metric_Pad0.98x0.95mm_HandSolder, symbol Device:R
- R2: value R -> 100R
- R3: value R -> 1k2
- R31: value R -> 1K
Connections:
- net GND: now also Q2.1 (E), R20.2; no longer R2.2
- net at J1.4 (RESET): now also R2.1
- net at R3.2: now also Q2.2 (B), R20.1
- new net: Q2.3 (C), R2.2
Other:
- note added: "TODO: Define these values based on testing TODO: Check grounding (don't connect wrong GNDs together)"
- note removed: "TODO: Define these values based on testing TODO: Add reset control TODO: Add +/- terminals to silkscreen TODO: Check grounding (don't connect wrong GNDs together)"
- moved on the sheet: R2
Changed lines of the file:
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@@
     (title "HD-Speccys")
     (date "2023-05-14")
-    (rev "1A")
+    (rev "1.0B")
     (company "RA Sewell")
   )
@@
   (junction (at 137.16 29.21) (diameter 0) (color 0 0 0 0)
   )
+  (junction (at 86.36 25.4) (diameter 0) (color 0 0 0 0)
+  )
   (junction (at 57.15 128.27) (diameter 0) (color 0 0 0 0)
   )
@@
   (junction (at 255.27 134.62) (diameter 0) (color 0 0 0 0)
   )
+  (junction (at 77.47 33.02) (diameter 0) (color 0 0 0 0)
+  )
   (junction (at 149.86 120.65) (diameter 0) (color 0 0 0 0)
   )
@@
     (stroke (width 0) (type default))
   )
-  (wire (pts (xy 88.9 35.56) (xy 88.9 39.37))
-    (stroke (width 0) (type default))
-  )
   (wire (pts (xy 259.08 71.12) (xy 255.27 71.12))
     (stroke (width 0) (type default))
@@
     (stroke (width 0) (type default))
   )
-  (wire (pts (xy 77.47 35.56) (xy 78.74 35.56))
-    (stroke (width 0) (type default))
-  )
   (wire (pts (xy 130.81 91.44) (xy 130.81 93.98))
     (stroke (width 0) (type default))
@@
     (stroke (width 0) (type default))
   )
-  (wire (pts (xy 64.77 39.37) (xy 64.77 17.78))
+  (wire (pts (xy 64.77 39.37) (xy 64.77 20.32))
     (stroke (width 0) (type default))
   )
@@
     (stroke (width 0) (type default))
   )
-  (wire (pts (xy 77.47 17.78) (xy 77.47 20.32))
-    (stroke (width 0) (type default))
-  )
   (wire (pts (xy 241.3 86.36) (xy 259.08 86.36))
     (stroke (width 0) (type default))
@@
     (stroke (width 0) (type default))
   )
-  (wire (pts (xy 77.47 30.48) (xy 77.47 35.56))
+  (wire (pts (xy 77.47 30.48) (xy 77.47 33.02))
     (stroke (width 0) (type default))
   )
@@
     (stroke (width 0) (type default))
   )
+  (wire (pts (xy 77.47 33.02) (xy 77.47 35.56))
+    (stroke (width 0) (type default))
+  )
   (wire (pts (xy 201.93 92.71) (xy 191.77 92.71))
     (stroke (width 0) (type default))
@@
     (stroke (width 0) (type default))
   )
+  (wire (pts (xy 64.77 20.32) (xy 67.31 20.32))
+    (stroke (width 0) (type default))
+  )
   (wire (pts (xy 35.56 77.47) (xy 57.15 77.47))
     (stroke (width 0) (type default))
@@
     (stroke (width 0) (type default))
   )
-  (wire (pts (xy 85.09 25.4) (xy 87.63 25.4))
+  (wire (pts (xy 85.09 25.4) (xy 86.36 25.4))
     (stroke (width 0) (type default))
   )
@@
     (stroke (width 0) (type default))
   )
+  (wire (pts (xy 86.36 25.4) (xy 87.63 25.4))
+    (stroke (width 0) (type default))
+  )
   (wire (pts (xy 115.57 140.97) (xy 115.57 118.11))
     (stroke (width 0) (type default))
@@
     (stroke (width 0) (type default))
   )
+  (wire (pts (xy 77.47 33.02) (xy 78.74 33.02))
+    (stroke (width 0) (type default))
+  )
   (wire (pts (xy 241.3 34.29) (xy 260.35 34.29))
     (stroke (width 0) (type default))
@@
     (stroke (width 0) (type default))
   )
+  (wire (pts (xy 86.36 33.02) (xy 86.36 25.4))
+    (stroke (width 0) (type default))
+  )
   (wire (pts (xy 35.56 128.27) (xy 57.15 128.27))
     (stroke (width 0) (type default))
@@
     (stroke (width 0) (type default))
   )
+  (wire (pts (xy 74.93 20.32) (xy 77.47 20.32))
+    (stroke (width 0) (type default))
+  )
   (wire (pts (xy 201.93 97.79) (xy 186.69 97.79))
     (stroke (width 0) (type default))
@@
     (stroke (width 0) (type default))
   )
-  (wire (pts (xy 64.77 17.78) (xy 77.47 17.78))
-    (stroke (width 0) (type default))
-  )
   (wire (pts (xy 30.48 172.72) (xy 30.48 177.8))
     (stroke (width 0) (type default))
@@
     (stroke (width 0) (type default))
   )
-  (wire (pts (xy 86.36 35.56) (xy 88.9 35.56))
-    (stroke (width 0) (type default))
-  )
   (wire (pts (xy 191.77 158.75) (xy 248.92 158.75))
     (stroke (width 0) (type default))
@@
     (stroke (width 0) (type default))
   )
-  (text "TODO: Define these values based on testing\nTODO: Add reset control\nTODO: Add +/- terminals to silkscreen\nTODO: Check grounding (don't connect wrong GNDs together)"
+  (text "TODO: Define these values based on testing\nTODO: Check grounding (don't connect wrong GNDs together)"
     (at 115.57 167.64 0)
     (effects (font (size 1.27 1.27)) (justify left bottom))
@@
     )
   )
-  (symbol (lib_id "Transistor_BJT:2N3906") (at 80.01 25.4 180) (unit 1)
-    (in_bom yes) (on_board yes) (dnp no)
-    (property "Reference" "Q1" (at 74.93 26.035 0)
-      (effects (font (size 1.27 1.27)) (justify left))
-    )
-    (property "Value" "2N3906" (at 74.93 23.495 0)
-      (effects (font (size 1.27 1.27)) (justify left))
-    )
-    (property "Footprint" "Package_TO_SOT_THT:TO-92_Inline" (at 74.93 23.495 0)
-      (effects (font (size 1.27 1.27) italic) (justify left) hide)
-    )
-    (property "Datasheet" "https://www.onsemi.com/pub/Collateral/2N3906-D.PDF" (at 80.01 25.4 0)
-      (effects (font (size 1.27 1.27)) (justify left) hide)
-    )
-    (pin "1")
-    (pin "2")
-    (pin "3")
-    (instances
-      (project "hd-speccys-1_0b"
-        (path "/d655584b-1b0c-4d69-832c-956bfbc09454"
-          (reference "Q1") (unit 1)
-        )
-      )
-    )
-  )
   (symbol (lib_id "Device:R") (at 171.45 158.75 270) (unit 1)
     (in_bom yes) (on_board yes) (dnp no) (fields_autoplaced)
@@
       (effects (font (size 1.27 1.27)))
     )
-    (property "Value" "R" (at 171.45 156.21 90)
+    (property "Value" "1K" (at 171.45 156.21 90)
       (effects (font (size 1.27 1.27)))
     )
@@
         (path "/d655584b-1b0c-4d69-832c-956bfbc09454"
           (reference "C2") (unit 1)
+        )
+      )
+    )
+  )
+  (symbol (lib_id "Transistor_BJT:2N3904") (at 80.01 25.4 0) (mirror y) (unit 1)
+    (in_bom yes) (on_board yes) (dnp no)
+    (property "Reference" "Q2" (at 74.93 24.765 0)
+      (effects (font (size 1.27 1.27)) (justify left))
+    )
+    (property "Value" "2N3904" (at 74.93 27.305 0)
+      (effects (font (size 1.27 1.27)) (justify left))
+    )
+    (property "Footprint" "Package_TO_SOT_THT:TO-92_Inline" (at 74.93 27.305 0)
+      (effects (font (size 1.27 1.27) italic) (justify left) hide)
+    )
+    (property "Datasheet" "https://www.onsemi.com/pub/Collateral/2N3903-D.PDF" (at 80.01 25.4 0)
+      (effects (font (size 1.27 1.27)) (justify left) hide)
+    )
+    (pin "1")
+    (pin "2")
+    (pin "3")
+    (instances
+      (project "hd-speccys-1_0b"
+        (path "/d655584b-1b0c-4d69-832c-956bfbc09454"
+          (reference "Q2") (unit 1)
         )
       )
@@
       (effects (font (size 1.27 1.27)))
     )
-    (property "Value" "R" (at 91.44 27.94 90)
-      (effects (font (size 1.27 1.27)) hide)
+    (property "Value" "1k2" (at 91.44 27.94 90)
+      (effects (font (size 1.27 1.27)))
     )
     (property "Footprint" "Resistor_SMD:R_0603_1608Metric_Pad0.98x0.95mm_HandSolder" (at 91.44 23.622 90)
@@
     )
   )
-  (symbol (lib_id "power:GND") (at 88.9 39.37 0) (unit 1)
-    (in_bom yes) (on_board yes) (dnp no) (fields_autoplaced)
-    (property "Reference" "#PWR03" (at 88.9 45.72 0)
-      (effects (font (size 1.27 1.27)) hide)
-    )
-    (property "Value" "GND" (at 88.9 44.45 0)
-      (effects (font (size 1.27 1.27)))
-    )
-    (property "Footprint" "" (at 88.9 39.37 0)
-      (effects (font (size 1.27 1.27)) hide)
-    )
-    (property "Datasheet" "" (at 88.9 39.37 0)
+  (symbol (lib_id "power:GND") (at 77.47 35.56 0) (unit 1)
+    (in_bom yes) (on_board yes) (dnp no) (fields_autoplaced)
+    (property "Reference" "#PWR03" (at 77.47 41.91 0)
+      (effects (font (size 1.27 1.27)) hide)
+    )
+    (property "Value" "GND" (at 77.47 40.64 0)
+      (effects (font (size 1.27 1.27)))
+    )
+    (property "Footprint" "" (at 77.47 35.56 0)
+      (effects (font (size 1.27 1.27)) hide)
+    )
+    (property "Datasheet" "" (at 77.47 35.56 0)
       (effects (font (size 1.27 1.27)) hide)
     )
@@
         (path "/d655584b-1b0c-4d69-832c-956bfbc09454"
           (reference "#PWR04") (unit 1)
+        )
+      )
+    )
+  )
+  (symbol (lib_id "Device:R") (at 82.55 33.02 270) (unit 1)
+    (in_bom yes) (on_board yes) (dnp no)
+    (property "Reference" "R20" (at 82.55 33.02 90)
+      (effects (font (size 1.27 1.27)))
+    )
+    (property "Value" "4K7" (at 82.55 35.56 90)
+      (effects (font (size 1.27 1.27)))
+    )
+    (property "Footprint" "Resistor_SMD:R_0603_1608Metric_Pad0.98x0.95mm_HandSolder" (at 82.55 31.242 90)
+      (effects (font (size 1.27 1.27)) hide)
+    )
+    (property "Datasheet" "~" (at 82.55 33.02 0)
+      (effects (font (size 1.27 1.27)) hide)
+    )
+    (pin "1")
+    (pin "2")
+    (instances
+      (project "hd-speccys-1_0b"
+        (path "/d655584b-1b0c-4d69-832c-956bfbc09454"
+          (reference "R20") (unit 1)
         )
       )
@@
     )
   )
-  (symbol (lib_id "Device:R") (at 82.55 35.56 90) (unit 1)
-    (in_bom yes) (on_board yes) (dnp no)
-    (property "Reference" "R2" (at 82.55 35.56 90)
-      (effects (font (size 1.27 1.27)))
-    )
-    (property "Value" "R" (at 82.55 33.02 90)
-      (effects (font (size 1.27 1.27)) hide)
-    )
-    (property "Footprint" "Resistor_SMD:R_0603_1608Metric_Pad0.98x0.95mm_HandSolder" (at 82.55 37.338 90)
-      (effects (font (size 1.27 1.27)) hide)
-    )
-    (property "Datasheet" "~" (at 82.55 35.56 0)
-      (effects (font (size 1.27 1.27)) hide)
-    )
+  (symbol (lib_id "Device:R") (at 71.12 20.32 90) (unit 1)
+    (in_bom yes) (on_board yes) (dnp no)
+    (property "Reference" "R2" (at 71.12 20.32 90)
+      (effects (font (size 1.27 1.27)))
+    )
+    (property "Value" "100R" (at 71.12 17.78 90)
+      (effects (font (size 1.27 1.27)))
+    )
+    (property "Footprint" "Resistor_SMD:R_0603_1608Metric_Pad0.98x0.95mm_HandSolder" (at 71.12 22.098 90)
+      (effects (font (size 1.27 1.27)) hide)
+    )
+    (property "Datasheet" "~" (at 71.12 20.32 0)
+      (effects (font (size 1.27 1.27)) hide)
+    )
